Commit message: goal 도착 이후의 구간을 계산해서 energy, eq_tracking cost를 추가함.

File: forestry_robot_mjcf/ecvt_v2_upper.urdf (robot description, URDF)
Before this commit: robot simple_model_for_urdf.SLDASM, 8 links, 7 joints
Links:
- link TOOL1: mass 467.870425947015 -> 467.87
- link UP1: mass 5233.6 -> 1089.36
- link UP2: mass 69.6789604825383 -> 546.98
- link UP3: mass 329.692051923496 -> 329.692
- link UP4: mass 195.721254726004 -> 195.721
- link UP5: mass 13.9596633124947 -> 13.9597
- link UP6: mass 71.3673205582859 -> 71.3673
- link base_link: mass 5233.6 -> 5233.5858073096

File: forestry_robot_mjcf/xml/ecvt_v2_upper.urdf (robot description, URDF)
Before this commit: robot simple_model_for_urdf.SLDASM, 8 links, 7 joints
Links:
- link TOOL1: mass 467.870425947015 -> 467.87
- link UP1: mass 5233.6 -> 1089.36
- link UP2: mass 69.6789604825383 -> 546.98
- link UP3: mass 329.692051923496 -> 329.692
- link UP4: mass 195.721254726004 -> 195.721
- link UP5: mass 13.9596633124947 -> 13.9597
- link UP6: mass 71.3673205582859 -> 71.3673
- link base_link: mass 5233.6 -> 5233.5858073096
Joints:
- joint UPJ5: type fixed -> revolute
- joint UPJ6: type fixed -> revolute
